File: hardware/Panel/Panel.kicad_pcb (KiCad board)
At the start: 2 copper layers, 100 x 200 mm, 22 parts

Commit message: Lots of updates belatedly committed
Parts:
- added G***: LOGO, Kosmo_panel:Quantizer_art, F.Cu at (100.0, 90.2)
- added H1: MountingHole, ao_tht:MountingHole_3.2mm_M3, F.Cu at (144.0, 90.0)
- added H2: MountingHole, ao_tht:MountingHole_3.2mm_M3, F.Cu at (144.0, 5.00)
- added H3: MountingHole, ao_tht:MountingHole_3.2mm_M3, F.Cu at (56.0, 90.0)
- added H4: MountingHole, ao_tht:MountingHole_3.2mm_M3, F.Cu at (56.0, 5.00)
