File: hardware/Panel components/quantpc.kicad_pcb (KiCad board)
At the start: 2 copper layers, 64 x 125 mm, 16 parts, among them J1 Conn_01x03 Scale_1, J2 Conn_01x03 Scale_2, J3 Conn_01x02 CV2_1, J4 Conn_01x02 CV2_2, J5 Conn_01x03 Bank_1, J6 Conn_01x03 Bank_2, J7 Conn_01x08, J8 Conn_01x04, J9 Conn_01x02, SW1 SW_SPST Quantize_1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

Commit message: Get rid of old daughterboard stuff
Parts:
- removed G***: LOGO, Daughterboard:analogoutput2
- removed H3, H4: MountingHole, MountingHole:MountingHole_3.2mm_M3
- removed J1: Conn_01x03 Scale_1, Connector_Molex:Molex_KK-254_AE-6410-03A_1x03_P2.54mm_Vertical
- removed J2: Conn_01x03 Scale_2, Connector_Molex:Molex_KK-254_AE-6410-03A_1x03_P2.54mm_Vertical
- removed J3: Conn_01x02 CV2_1, Connector_Molex:Molex_KK-254_AE-6410-02A_1x02_P2.54mm_Vertical
- removed J4: Conn_01x02 CV2_2, Connector_Molex:Molex_KK-254_AE-6410-02A_1x02_P2.54mm_Vertical
- removed J5: Conn_01x03 Bank_1, Connector_Molex:Molex_KK-254_AE-6410-03A_1x03_P2.54mm_Vertical
- removed J6: Conn_01x03 Bank_2, Connector_Molex:Molex_KK-254_AE-6410-03A_1x03_P2.54mm_Vertical
- removed J7: Conn_01x08, Connector_PinSocket_2.54mm:PinSocket_1x08_P2.54mm_Vertical
- removed J8: Conn_01x04, Connector_PinSocket_2.54mm:PinSocket_1x04_P2.54mm_Vertical
- removed J9: Conn_01x02, Connector_PinSocket_2.54mm:PinSocket_1x02_P2.54mm_Vertical
- removed RV1, RV2: 10k, Potentiometer_THT:Potentiometer_Alpha_RD901F-40-00D_Single_Vertical_CircularHoles
- removed SW1: SW_SPST Quantize_1, Daughterboard:SPDT-toggle-switch-1M-series
- removed SW2: SW_SPST Quantize_2, Daughterboard:SPDT-toggle-switch-1M-series
Routing:
- net Net-(J3-Pad1): track 109.0 -> 0.00 mm
- net Net-(J1-Pad2): track 73.2 -> 0.00 mm
- net Net-(J2-Pad2): track 65.7 -> 0.00 mm
- net Net-(J5-Pad2): track 63.9 -> 0.00 mm
- net Net-(J6-Pad2): track 58.9 -> 0.00 mm
- net Net-(J9-Pad1): track 51.3 -> 0.00 mm
- net VCC: track 49.1 -> 0.00 mm
- net Net-(J7-Pad4): track 48.1 -> 0.00 mm
- net Net-(J4-Pad1): track 45.5 -> 0.00 mm
- net Net-(J9-Pad2): track 31.7 -> 0.00 mm
- net Net-(J7-Pad2): track 20.0 -> 0.00 mm
- removed copper zone on B.Cu, net GND
- removed copper zone on F.Cu, net GND
Other:
- board outline removed
- board text removed: "Bank 1"
- board text removed: "Bank 2"
- board text removed: "CV2 1"
- board text removed: "CV2 2"
- board text removed: "Dual Quantizer Rich Holmes May 2020"
- board text removed: "Scale 1"
- board text removed: "Scale 2"
